File: Boards/mainBoard/Nixie_v1.kicad_sch (KiCad schematic)
At the start: 66 parts

Commit message: Remove unused symbols from Schematic
Parts:
- removed #ENC1: (no value), symbol Nixie_v1-eagle-import:ROTARY-ENCODER_OFF-BOARD
- removed #POT1: (no value), symbol Nixie_v1-eagle-import:POT_OFF-BOARD
- removed #S3, #S4, #S5: (no value), symbol Nixie_v1-eagle-import:SPST_OFF-BOARD
- removed C10, C11, C7, C8, C9: (no value), symbol Nixie_v1-eagle-import:C2.5/2
- removed IC10, IC11, IC12, IC13, IC8, IC9: (no value), symbol Nixie_v1-eagle-import:LED-RGB_CLY6D-FKC-CK1N1D1BB7D3D3
- removed J2: (no value), symbol Nixie_v1-eagle-import:CONNECTOR_6PINSCREW_TERMINAL_5MM_PITCH
- removed J3: (no value), symbol Nixie_v1-eagle-import:CONNECTOR_4PIN
- removed J4: (no value), symbol Nixie_v1-eagle-import:CONNECTOR_5PIN
- removed Q1: (no value), symbol Nixie_v1-eagle-import:XTAL/S
- removed R10, R11, R12, R13, R14, R15, R16, R17, R18, R19, R20, R9: (no value), symbol Nixie_v1-eagle-import:R-US_0207/7
- removed S1: (no value), symbol Nixie_v1-eagle-import:MOMENTARY-SWITCH-SPST-PTH-6.0MM
- #S2: value (none) -> SPDT-LED_OFF-BOARD; footprint (none) -> Nixie_v1:
- C1, C12, C2, C3, C4, C5, C6: value (none) -> 0.1uF; footprint (none) -> Nixie_v1:C2.5-2
- IC1, IC2, IC3, IC4, IC5, IC6: value (none) -> TPIC6595N; footprint (none) -> Nixie_v1:DIP20
- IC7: value (none) -> PIC16F15325; footprint (none) -> Nixie_v1:DIP14
- J1: value (none) -> Screw Terminal 4 Pin; footprint (none) -> Nixie_v1:SCREW_TERM_5MM_1X4
- NB1, NB2: value (none) -> IN-3; footprint (none) -> Nixie_v1:IN-3
- NX1, NX2, NX3, NX4, NX5, NX6: value (none) -> NIXIE_IN-12A; footprint (none) -> Nixie_v1:IN-12_NO_HOLE
- R1, R2, R3, R4, R5, R6: value (none) -> 14k; footprint (none) -> Nixie_v1:0411_12
- R7, R8: value (none) -> 162k; footprint (none) -> Nixie_v1:0411_12
- SYM101: value (none) -> SYMBOL_HIGH_VOLTAGE; footprint (none) -> Nixie_v1:SYMBOL_HIGH_VOLTAGE
Other:
- note added: "Total Current Draw from Wall Power Using +12V for Nixie Power Supply Nixies OFF: 15mA Nixies ON: 270mA Use a 0.5 Amp PTC Fuse"
- note removed: "Latching SPST Switches to control RGB LEDs 1k POT as a Dimmer ***ALL EXTERNAL***"
- note removed: "Rotary Encoder (RPG) for "User Set" mode to set the clock. Encoder has a PB switch integrated to switch bewtween setting HH,MM,SS and "Free Running". ***EXTERNAL***"
- note removed: "Total Current Draw from Wall Power Using +12V for Nixie Power Supply Nixies OFF, LEDs OFF: 15mA Nixies ON, LEDs OFF: 270mA Nixies ON, R LED ON: 294mA Nixies ON, G LED ON: 290mA Nixies ON, B LED ON: 296mA Nixies ON, RGB LED ON: 340mA Use a 0.5 Amp PTC Fuse"
- note removed: "Vred = 2.1V Vgreen = 2.7V Vblue = 3.0V Want 10mA max per LED With 12V supply Ideal Resistors Rred = 570 Rgreen = 390 Rblue = 300"
- note removed: "~{MCLR VDD VSS PGD PGC}"
